Commit message: add 2rov

File: src/uuv_simulator/uuv_sensor_plugins/uuv_sensor_ros_plugins/urdf/pressure_snippets.xacro (robot description, xacro)
@@ -39,5 +39,5 @@
     </xacro:pressure_plugin_macro>
   </xacro:macro>
-  <xacro:macro name="default_pressure" params="namespace parent_link *origin">
+  <!-- <xacro:macro name="default_pressure" params="namespace parent_link *origin">
     <xacro:pressure_plugin_macro
       namespace="${namespace}"
@@ -56,5 +56,5 @@
       <xacro:insert_block name="origin" />
     </xacro:pressure_plugin_macro>
-  </xacro:macro>
+  </xacro:macro> -->
   <xacro:macro name="pressure_plugin_macro"
     params="namespace suffix parent_link topic mass update_rate
